File: hackpad/_restore_backup_2026-08-29T14-43-20-922/hackpad.kicad_pcb (KiCad board)
At the start: 2 copper layers, 63.7 x 78.7 mm, 15 parts, among them SW1 SW_Push, SW10 SW_Push, SW2 SW_Push, SW3 SW_Push, SW4 SW_Push, SW5 SW_Push, SW6 SW_Push, SW7 SW_Push, SW9 SW_Push, U1 MOUDLE-SEEEDUINO-XIAO

Commit message: Finished PCB
Parts:
- moved U2 3.66 mm to (155.0, 51.0)
Routing:
- net /OLED SCL: track 14.0 -> 6.32 mm
- net /<NO NET>: track 5.50 -> 10.9 mm
- net Net-(D1-DIN): track 51.9 -> 47.4 mm
- net GND: track 190.1 -> 192.0 mm
- net /LED VDD: track 140.3 -> 141.9 mm
- net /OLED VCC: track 21.8 -> 21.0 mm
